File: _autosave-DashMotor48V.kicad_pcb (KiCad board)
At the start: 4 copper layers, 71.8 x 70.7 mm, 79 parts, among them CN3(OUT)1 XT30(2+2)PB-M.G.B, CN3(OUT)2 XT30(2+2)PB-M.G.B, J1 BM07B-SRSS-TB, J2 BM07B-SRSS-TB, Q1 FDMS039N08B, Q2 FDMS039N08B, Q3 FDMS039N08B, Q4 FDMS039N08B, Q5 FDMS039N08B, Q6 FDMS039N08B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

Commit message: get the footprint for the bigger motor
Parts:
- moved Q1 60.8 mm to (184.6, 74.5)
- moved Q3 60.8 mm to (191.6, 74.5)
- moved Q5 60.8 mm to (198.6, 74.5)
- moved H1 59.6 mm to (184.9, 67.0)
- moved H2 59.6 mm to (191.9, 67.0)
- moved H3 59.6 mm to (198.9, 67.0)
- moved Q2 59.6 mm to (184.9, 59.5)
- moved Q4 59.6 mm to (191.9, 59.5)
- moved Q6 59.6 mm to (198.9, 59.5)
- moved J1 42.2 mm to (137.7, 118.6)
- moved J2 42.2 mm to (137.7, 126.0)
- moved CN3(OUT)1 28.2 mm to (155.5, 120.1)
- moved CN3(OUT)2 18.3 mm to (217.0, 120.1)
Changed lines of the file:
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@@
 	(footprint "MountingHole:MountingHole_2.2mm_M2_Pad"
 		(layer "F.Cu")
-		(at 233.8 101.2)
+		(at 184.935 67.03)
 		(descr "Mounting Hole 2.2mm, M2, generated by kicad-footprint-generator mountinghole.py")
 		(tags "mountinghole M2")
@@
 	(footprint "dash:FDMS039N08B"
 		(layer "F.Cu")
-		(at 233.8 93.7 180)
+		(at 184.935 59.53 180)
 		(descr "PQFN8 5X6, 1.27P CASE 483AE ISSUE A_1")
 		(tags "MOSFET (N-Channel)")
@@
 	(footprint "dash:FDMS039N08B"
 		(layer "F.Cu")
-		(at 241.4 109.4 180)
+		(at 191.635 74.472 180)
 		(descr "PQFN8 5X6, 1.27P CASE 483AE ISSUE A_1")
 		(tags "MOSFET (N-Channel)")
@@
 	(footprint "dash:FDMS039N08B"
 		(layer "F.Cu")
-		(at 248.4 109.4 180)
+		(at 198.635 74.472 180)
 		(descr "PQFN8 5X6, 1.27P CASE 483AE ISSUE A_1")
 		(tags "MOSFET (N-Channel)")
@@
 	(footprint "MountingHole:MountingHole_2.2mm_M2_Pad"
 		(layer "F.Cu")
-		(at 240.8 101.2)
+		(at 191.935 67.03)
 		(descr "Mounting Hole 2.2mm, M2, generated by kicad-footprint-generator mountinghole.py")
 		(tags "mountinghole M2")
@@
 	(footprint "dash:XT30(2+2)PB-M.G.B"
 		(layer "F.Cu")
-		(at 127.3 120.924999 90)
+		(at 155.5 120.075 90)
 		(property "Reference" "CN3(OUT)1"
 			(at -0.2 -3.427 90)
@@
 	(footprint "dash:FDMS039N08B"
 		(layer "F.Cu")
-		(at 247.8 93.7 180)
+		(at 198.935 59.53 180)
 		(descr "PQFN8 5X6, 1.27P CASE 483AE ISSUE A_1")
 		(tags "MOSFET (N-Channel)")
@@
 	(footprint "dash:FDMS039N08B"
 		(layer "F.Cu")
-		(at 240.8 93.7 180)
+		(at 191.935 59.53 180)
 		(descr "PQFN8 5X6, 1.27P CASE 483AE ISSUE A_1")
 		(tags "MOSFET (N-Channel)")
@@
 	(footprint "dash:BM07B-SRSS-TB"
 		(layer "F.Cu")
-		(at 96.000001 132.5784)
+		(at 137.699998 125.9511)
 		(tags "BM07B-SRSS-TB ")
 		(property "Reference" "J2"
@@
 	(footprint "MountingHole:MountingHole_2.2mm_M2_Pad"
 		(layer "F.Cu")
-		(at 247.8 101.2)
+		(at 198.935 67.03)
 		(descr "Mounting Hole 2.2mm, M2, generated by kicad-footprint-generator mountinghole.py")
 		(tags "mountinghole M2")
@@
 	(footprint "dash:XT30(2+2)PB-M.G.B"
 		(layer "F.Cu")
-		(at 235 123.175002 -90)
+		(at 217 120.075002 -90)
 		(property "Reference" "CN3(OUT)2"
 			(at -0.2 -3.427 90)
@@
 	(footprint "dash:BM07B-SRSS-TB"
 		(layer "F.Cu")
-		(at 96.000001 125.230699)
+		(at 137.699998 118.603399)
 		(tags "BM07B-SRSS-TB ")
 		(property "Reference" "J1"
@@
 	(footprint "dash:FDMS039N08B"
 		(layer "F.Cu")
-		(at 234.4 109.4 180)
+		(at 184.635 74.472 180)
 		(descr "PQFN8 5X6, 1.27P CASE 483AE ISSUE A_1")
 		(tags "MOSFET (N-Channel)")
