File: v0.5/DashMotor48V.kicad_pcb (KiCad board)
At the start: 6 copper layers, 72 x 69.7 mm, 114 parts, among them CN3(OUT)1 XT30(2+2)PB-M.G.B, CN3(OUT)2 XT30(2+2)PB-M.G.B, J1 BM07B-SRSS-TB(LF)(SN), J2 BM07B-SRSS-TB(LF)(SN), Q1 FDMT80080DC, Q2 FDMT80080DC, Q3 FDMT80080DC, Q4 FDMT80080DC, Q5 FDMT80080DC, Q6 FDMT80080DC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

Commit message: upload again
Parts:
- removed C25, C27, C32, C46: CL31B105KCHNNNE, dash:CL31B105KCHNNNE
- added C22: 1uF 100V, dash:GRM21BC72A105KE01L, F.Cu at (-8.51, -23.8)
- added C28: 1uF 100V, dash:GRM21BC72A105KE01L, F.Cu at (-8.01, -10.3)
- added C29: 1uF 100V, dash:GRM21BC72A105KE01L, F.Cu at (-6.01, -10.3)
- added C30: 1uF 100V, dash:GRM21BC72A105KE01L, B.Cu at (-1.27, 3.51)
- moved Q2 0.70 mm to (-14.5, 11.0)
- moved Q5 0.70 mm to (14.5, 11.0)
- moved Q1 0.50 mm to (-24.5, 5.00)
- moved Q6 0.50 mm to (24.5, 5.00)
- moved Q3 0.40 mm to (5.00, 15.0)
- moved Q4 0.40 mm to (-5.00, 15.0)

Commit message: work on routing
Parts:
- moved R16 2.25 mm to (-12.0, 2.50)
- moved R18 0.98 mm to (13.0, 2.50)
- moved C18 0.95 mm to (18.2, 3.50)
- moved C8 0.91 mm to (-18.2, 3.50)
- moved C51 0.72 mm to (-6.65, -5.00), turned to 180 degrees
- moved H1 0.50 mm to (-14.5, 24.0)
- moved H3 0.50 mm to (14.5, 24.0)
- moved C14 0.40 mm to (27.5, -0.50)
- moved C15 0.20 mm to (23.9, -0.50)
- moved C16 0.19 mm to (17.0, 7.70)
- moved C13 0.16 mm to (13.6, 7.70)
- moved C4 0.13 mm to (-13.6, 7.70)
- moved C12 0.12 mm to (10.2, 7.70)
- moved C7 0.12 mm to (6.80, 7.70)
- moved C6 0.11 mm to (-6.80, 7.70)
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Routing:
- net /GHA: track 34.1 -> 0.00 mm
- net /PHASC: track 27.9 -> 24.8 mm
- net /PHASB: track 23.7 -> 22.6 mm
- net /GLA: track 15.2 -> 16.0 mm
- net /GLC: track 32.0 -> 32.6 mm
- added copper zone on F.Cu, net /PHASA
- added copper zone on F.Cu, net /PHASB
- added copper zone on F.Cu, net /PHASC

Commit message: push
Parts:
- moved C11 6.44 mm to (-18.2, -3.50), turned to 180 degrees
- moved C15 6.44 mm to (18.2, -3.50), turned to 0 degrees
- moved C10 4.53 mm to (-23.0, 0.00), turned to 0 degrees
- moved C14 4.53 mm to (23.0, 0.00), turned to 180 degrees
- moved C17 2.16 mm to (18.2, 0.00), turned to 0 degrees
- moved C19 2.16 mm to (-18.2, 0.00), turned to 180 degrees
- moved CC1 0.61 mm to (-19.0, -7.00)
- moved CC2 0.61 mm to (19.0, -7.00)
- moved Q1 0.50 mm to (-24.5, 5.50)
- moved Q6 0.50 mm to (24.5, 5.50)
Routing:
- net GND: track 19.9 -> 17.7 mm
- added copper zone on B.Cu, net +48V
- added copper zone on B.Cu, net GND
- removed copper zone on In2.Cu, net +12V

Commit message: push
Parts:
- moved VR1 53.1 mm to (-63.0, -20.6), turned to 90 degrees
- moved C37 50.5 mm to (-64.1, -13.1)
- moved C42 33.3 mm to (-40.9, -18.2)
- moved L1 32.3 mm to (-46.9, -25.6)
- moved R14 24.9 mm to (-33.5, -13.3)
- moved R15 22.8 mm to (-34.1, -15.7)
- moved R13 19.3 mm to (-29.1, -19.1)
- moved C38 17.9 mm to (-29.4, -15.9)
- moved C43 17.2 mm to (-28.7, -13.4)
- moved R9 16.8 mm to (-26.0, -16.8)
- moved C39 14.5 mm to (-28.2, -26.8)
Routing:
- net /GHA: track 0.00 -> 32.8 mm
- net /PHASA: track 29.1 -> 25.9 mm, vias 0 -> 18
- net /GLC: track 32.6 -> 29.7 mm
- net /SPC: track 17.1 -> 14.8 mm
- net /PWMC: track 8.12 -> 6.28 mm
- net /PHASB: track 22.6 -> 20.8 mm, vias 0 -> 18
- net /SPB: track 12.5 -> 10.9 mm
- net /GLB: track 17.5 -> 16.0 mm
- net /PWMB: track 6.54 -> 5.24 mm
- net /GHB: track 26.2 -> 25.0 mm
- net /GHC: track 23.9 -> 22.7 mm
- net /SPA: track 21.6 -> 20.6 mm
- net /GLA: track 16.0 -> 15.0 mm
- net /PHASC: track 24.8 -> 25.6 mm, vias 0 -> 18
- net +48V: vias 32 -> 122
- added copper zone on F.Cu, net /SPA
- added copper zone on F.Cu, net /SPB
- added copper zone on F.Cu, net /SPC

Commit message: backup
Parts:
- C37, L1: moved to F.Cu
- moved VR1 45.5 mm to (-18.9, -9.15)
- moved C39 28.2 mm to (-43.5, -3.15), turned to 180 degrees
- moved C38 25.8 mm to (-51.5, -2.65), turned to 0 degrees
- moved L1 24.5 mm to (-46.5, -1.15), turned to 90 degrees
- moved R9 21.8 mm to (-45.0, -6.15), turned to 90 degrees
- moved C42 20.7 mm to (-54.5, -2.65), turned to 180 degrees
- moved C43 20.6 mm to (-47.5, -5.15), turned to 0 degrees
- moved R15 19.9 mm to (-51.0, -5.15)
- moved C37 19.8 mm to (-53.0, 3.35), turned to -90 degrees
- moved R14 15.4 mm to (-47.5, -7.15), turned to 0 degrees
- moved R13 13.1 mm to (-23.0, -7.50), turned to -90 degrees
- moved TP1 10.6 mm to (-38.0, -14.0)
- moved R1 7.83 mm to (-17.5, -16.5)
- moved TP_GND1 7.03 mm to (-42.0, -20.5)
- moved R3 3.46 mm to (-14.5, -23.0)
Routing:
- net GND: track 17.7 -> 11.3 mm
- net /SPI-MOSI: track 1.69 -> 0.00 mm
- added copper zone on In2.Cu, net +48V

Commit message: backup
Parts:
- C20: moved to F.Cu
- C37, L1: moved to B.Cu
- moved C42 49.3 mm to (-6.57, -14.2), turned to 0 degrees
- moved R9 38.8 mm to (-6.60, -11.6)
- moved L1 38.3 mm to (-10.6, -14.4), turned to -90 degrees
- moved R14 36.6 mm to (-12.8, -18.6), turned to 180 degrees
- moved R15 36.2 mm to (-15.8, -13.2), turned to 90 degrees
- moved C38 35.2 mm to (-18.2, -14.0)
- moved C43 34.3 mm to (-14.2, -13.2), turned to -90 degrees
- moved C37 30.6 mm to (-23.2, -3.40), turned to 0 degrees
- moved C39 29.8 mm to (-14.4, -9.20), turned to 0 degrees
- moved C20 7.89 mm to (-11.2, -3.80), turned to 180 degrees
- moved C21 4.65 mm to (-10.0, -8.00)
- moved C51 1.57 mm to (-5.20, -4.40), turned to -90 degrees
- moved R13 1.36 mm to (-23.8, -6.40), turned to 0 degrees
- moved VR1 0.50 mm to (-19.4, -9.15)
Routing:
- net Net-(VR1-FB): track 0.00 -> 14.3 mm
- net Net-(VR1-SW): track 0.00 -> 11.9 mm
- net Net-(C42-Pad1): track 0.00 -> 8.87 mm
- net Net-(VR1-BST): track 0.00 -> 2.21 mm

Commit message: keep routing
Parts:
- removed R1: RC0402FR-07150KL, dash:RC0402FR_07150KL
- added R6: YAGEO RC0603FR-07200KL, dash:YAGEO RC0603FR-07200KL, F.Cu at (37.8, 19.0)
Routing:
- net +48V: vias 122 -> 138
- added copper zone on F.Cu, net +48V

Commit message: keep routing
Parts:
- removed C31: 100nF 50V, dash:CC0603JRX7R9BB104
- added C57: 100nF 100V, dash:CL10B104KC8NNNC, F.Cu at (8.25, -24.0)
- added J3: Conn_01x02_Pin, Connector_PinHeader_2.54mm:PinHeader_1x02_P2.54mm_Vertical, F.Cu at (-20.6, -19.1)
- C24, FL1, Y1: moved to B.Cu
- U3: moved to F.Cu
- moved R6 56.6 mm to (-12.6, -6.66), turned to 90 degrees
- moved C55 23.7 mm to (-13.2, -16.0), turned to 180 degrees
- moved C52 7.96 mm to (18.0, -21.1), turned to 0 degrees
- moved R12 7.72 mm to (13.9, -13.7)
- moved R2 7.57 mm to (-11.1, -15.9), turned to 90 degrees
- moved U3 7.44 mm to (17.6, -18.2)
- moved L3 6.94 mm to (19.8, -17.0), turned to 180 degrees
- moved Y1 6.48 mm to (3.02, -22.6)
- moved C41 5.47 mm to (16.1, -18.0), turned to -90 degrees
- moved R8 3.91 mm to (-15.6, -18.5)
- moved D2 3.91 mm to (-15.6, -15.8)
- moved R7 3.91 mm to (-17.2, -18.5)
- moved C53 3.87 mm to (13.8, -18.4), turned to 90 degrees
- moved D1 3.86 mm to (-17.2, -15.8)
- moved R5 3.66 mm to (-7.38, -31.2)
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Connections:
- CN3(OUT)1 pad 1: /CAN+ -> /CAN-
- CN3(OUT)1 pad 2: /CAN- -> /CAN+
- CN3(OUT)2 pad 1: /CAN+ -> /CAN-
- CN3(OUT)2 pad 2: /CAN- -> /CAN+
- U1 pad 10: /I_C -> /I_A
- U1 pad 8: /I_A -> /I_C
Routing:
- net /CAN+: track 0.00 -> 77.3 mm, vias 0 -> 1
- net /CAN-: track 0.62 -> 76.7 mm, vias 0 -> 1
- net +3.3V: track 6.25 -> 61.5 mm, vias 1 -> 5
- net /SCK: track 11.1 -> 46.6 mm, vias 1 -> 3
- net /MISO: track 10.9 -> 44.3 mm, vias 1 -> 3
- net /MOSI: track 11.4 -> 44.0 mm, vias 1 -> 3
- net /VMOT_TEMP: track 0.00 -> 29.0 mm, vias 0 -> 1
- net /TCK: track 3.82 -> 30.5 mm, vias 0 -> 2
- net +5V: track 0.00 -> 25.1 mm, vias 0 -> 1
- net /CS: track 0.00 -> 24.0 mm, vias 0 -> 2
- net +12V: track 0.00 -> 23.7 mm, vias 0 -> 1
- net /I_C: track 0.00 -> 23.2 mm, vias 0 -> 2
- net /SPI-NSS-DRV: track 0.00 -> 23.0 mm, vias 0 -> 2
- net /VBAT: track 0.00 -> 22.7 mm, vias 0 -> 2
- net /I_B: track 0.00 -> 22.3 mm, vias 0 -> 2
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- added copper zone on B.Cu, net +12V
- added copper zone on B.Cu, net +3.3V
- added copper zone on B.Cu, net +5V
