File: v0.5/DashMotor48V.kicad_pcb (KiCad board)
At the start: 6 copper layers, 72 x 69.7 mm, 108 parts, among them CN3(OUT)1 XT30(2+2)PB-M.G.B, CN3(OUT)2 XT30(2+2)PB-M.G.B, J1 BM07B-SRSS-TB(LF)(SN), J2 BM07B-SRSS-TB(LF)(SN), J3 Conn_01x02_Pin, Q1 FDMT80080DC, Q2 FDMT80080DC, Q3 FDMT80080DC, Q4 FDMT80080DC, Q5 FDMT80080DC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

Commit message: finetuning
Parts:
- moved C16 0.50 mm to (16.5, 7.70)
- moved C9 0.50 mm to (-16.5, 7.70)
- moved C13 0.40 mm to (13.2, 7.70)
- moved C4 0.40 mm to (-13.2, 7.70)
- moved C12 0.30 mm to (9.90, 7.70)
- moved C5 0.30 mm to (-9.90, 7.70)
- moved C6 0.20 mm to (-6.60, 7.70)
- moved C7 0.20 mm to (6.60, 7.70)
- moved C1 0.10 mm to (-3.30, 7.70)
- moved C3 0.10 mm to (3.30, 7.70)
Routing:
- net GND: track 71.5 -> 71.4 mm, vias 113 -> 194
- net /PHASC: vias 32 -> 74
- net /PHASB: vias 32 -> 74
- net /PHASA: vias 32 -> 74
- net +48V: vias 150 -> 260
