File: v0.5/DashMotor48V.kicad_sch (KiCad schematic)
At the start: 110 parts, among them CN3(OUT)1 XT30(2+2)PB-M.G.B, CN3(OUT)2 XT30(2+2)PB-M.G.B, J1 BM07B-SRSS-TB(LF)(SN), J2 BM07B-SRSS-TB(LF)(SN), J3 Conn_01x02_Pin, Q1 FDMT80080DC, Q2 FDMT80080DC, Q3 FDMT80080DC, Q4 FDMT80080DC, Q5 FDMT80080DC, Q6 FDMT80080DC, U1 STM32F446RET6, U2 DRV8353SRTAR, U3 MCP2542FD-E/MF, U4 MA732GQ-Z, U5 TPS629203DRLR, U6 TPS629203DRLR, Y1 CSTNE8M00G550000R0

Commit message: keep finishing it
Parts:
- removed TP1: +12V TestPoint, TestPoint:TestPoint_THTPad_D1.5mm_Drill0.7mm, symbol Connector:TestPoint
- TP10, TP7, TP8, TP9: footprint TestPoint:TestPoint_THTPad_D1.0mm_Drill0.5mm -> TestPoint:TestPoint_Pad_D1.0mm
- TP4: footprint TestPoint:TestPoint_THTPad_D1.5mm_Drill0.7mm -> TestPoint:TestPoint_Pad_D1.0mm
Changed lines of the file:
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@@
 	)
 	(junction
-		(at 151.13 299.72)
-		(diameter 0)
-		(color 0 0 0 0)
-	)
-	(junction
 		(at 156.21 152.4)
 		(diameter 0)
@@
 	(wire
 		(pts
-			(xy 146.05 299.72) (xy 151.13 299.72)
+			(xy 146.05 299.72) (xy 157.48 299.72)
 		)
 		(stroke
@@
 	(wire
 		(pts
-			(xy 151.13 299.72) (xy 157.48 299.72)
-		)
-		(stroke
-			(width 0)
-			(type default)
-		)
-	)
-	(wire
-		(pts
 			(xy 215.9 161.29) (xy 215.9 163.83)
 		)
@@
 			)
 		)
-		(property "Footprint" "TestPoint:TestPoint_THTPad_D1.0mm_Drill0.5mm"
+		(property "Footprint" "TestPoint:TestPoint_Pad_D1.0mm"
 			(at 254 130.81 0)
 			(hide yes)
@@
 	)
 	(symbol
-		(lib_id "Connector:TestPoint")
-		(at 151.13 299.72 180)
-		(unit 1)
-		(body_style 1)
-		(exclude_from_sim no)
-		(in_bom yes)
-		(on_board yes)
-		(in_pos_files yes)
-		(dnp no)
-		(fields_autoplaced yes)
-		(property "Reference" "TP1"
-			(at 153.67 301.7519 0)
-			(show_name no)
-			(do_not_autoplace no)
-			(effects
-				(font
-					(size 1.27 1.27)
-				)
-				(justify right)
-			)
-		)
-		(property "Value" "+12V TestPoint"
-			(at 153.67 304.2919 0)
-			(show_name no)
-			(do_not_autoplace no)
-			(effects
-				(font
-					(size 1.27 1.27)
-				)
-				(justify right)
-			)
-		)
-		(property "Footprint" "TestPoint:TestPoint_THTPad_D1.5mm_Drill0.7mm"
-			(at 146.05 299.72 0)
-			(hide yes)
-			(show_name no)
-			(do_not_autoplace no)
-			(effects
-				(font
-					(size 1.27 1.27)
-				)
-			)
-		)
-		(property "Datasheet" ""
-			(at 146.05 299.72 0)
-			(hide yes)
-			(show_name no)
-			(do_not_autoplace no)
-			(effects
-				(font
-					(size 1.27 1.27)
-				)
-			)
-		)
-		(property "Description" "test point"
-			(at 151.13 299.72 0)
-			(hide yes)
-			(show_name no)
-			(do_not_autoplace no)
-			(effects
-				(font
-					(size 1.27 1.27)
-				)
-			)
-		)
-		(pin "1"
-		)
-		(instances
-			(project "DashMotor48V"
-				(path "/71f0fcc1-c7ad-470c-8d48-d038c53969d3"
-					(reference "TP1")
-					(unit 1)
-				)
-			)
-		)
-	)
-	(symbol
 		(lib_id "power:GND")
 		(at 237.49 271.78 0)
@@
 			)
 		)
-		(property "Footprint" "TestPoint:TestPoint_THTPad_D1.0mm_Drill0.5mm"
+		(property "Footprint" "TestPoint:TestPoint_Pad_D1.0mm"
 			(at 200.66 125.73 0)
 			(hide yes)
@@
 			)
 		)
-		(property "Footprint" "TestPoint:TestPoint_THTPad_D1.0mm_Drill0.5mm"
+		(property "Footprint" "TestPoint:TestPoint_Pad_D1.0mm"
 			(at 254 140.97 0)
 			(hide yes)
@@
 			)
 		)
-		(property "Footprint" "TestPoint:TestPoint_THTPad_D1.5mm_Drill0.7mm"
+		(property "Footprint" "TestPoint:TestPoint_Pad_D1.0mm"
 			(at 379.73 313.69 0)
 			(hide yes)
@@
 			)
 		)
-		(property "Footprint" "TestPoint:TestPoint_THTPad_D1.0mm_Drill0.5mm"
+		(property "Footprint" "TestPoint:TestPoint_Pad_D1.0mm"
 			(at 254 135.89 0)
 			(hide yes)
