File: v0.5/DashMotor48V.kicad_sch (KiCad schematic)
At the start: 109 parts, among them CN3(OUT)1 XT30(2+2)PB-M.G.B, CN3(OUT)2 XT30(2+2)PB-M.G.B, J1 BM07B-SRSS-TB(LF)(SN), J2 BM07B-SRSS-TB(LF)(SN), J3 Conn_01x02_Pin, Q1 FDMT80080DC, Q2 FDMT80080DC, Q3 FDMT80080DC, Q4 FDMT80080DC, Q5 FDMT80080DC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

Commit message: doing fine touch for the routing, almost done
Parts:
- removed TP11: TP_MOSI, TestPoint:TestPoint_THTPad_D1.0mm_Drill0.5mm, symbol Connector:TestPoint
- removed TP13: TP_MISO, TestPoint:TestPoint_THTPad_D1.0mm_Drill0.5mm, symbol Connector:TestPoint
- removed TP14: TP_SCK, TestPoint:TestPoint_THTPad_D1.0mm_Drill0.5mm, symbol Connector:TestPoint
Other:
- moved on the sheet: C56, J3, R5
